File: PCB/MainBoard.kicad_pcb (KiCad board)
At the start: 2 copper layers, 302.5 x 158.3 mm, 15 parts, among them U2 ATmega2560-16A, Y1 Crystal_GND24

Commit message: Worked on schematic, added USB-C, worked on pcb
Parts:
- removed C1, C2: 22p, Capacitor_SMD:C_0603_1608Metric
- removed U2: ATmega2560-16A, Package_QFP:TQFP-100_14x14mm_P0.5mm
- removed Y1: Crystal_GND24, Crystal:Crystal_SMD_SeikoEpson_FA238-4Pin_3.2x2.5mm
- added C10: 22p, Capacitor_SMD:C_0603_1608Metric, F.Cu at (263.2, 45.0)
- added C11: 1u, Capacitor_SMD:C_0603_1608Metric, F.Cu at (98.8, 94.8)
- added C8: 22p, Capacitor_SMD:C_0603_1608Metric, F.Cu at (267.2, 45.0)
- added J1: USB4105-GF-A, USB4105_GF_A:GCT_USB4105-GF-A, F.Cu at (259.7, 19.5)
- added R10: 5.1k, Resistor_SMD:R_0603_1608Metric, F.Cu at (98.8, 109.8)
- added R2: 22, Resistor_SMD:R_0603_1608Metric, F.Cu at (98.8, 97.3)
- added R3: 22, Resistor_SMD:R_0603_1608Metric, F.Cu at (98.8, 99.8)
- added R6: 10k, Resistor_SMD:R_0603_1608Metric, F.Cu at (98.8, 102.3)
- added R7: 10k, Resistor_SMD:R_0603_1608Metric, F.Cu at (98.8, 104.8)
- added R9: 5.1k, Resistor_SMD:R_0603_1608Metric, F.Cu at (98.8, 107.3)
- added SW_RESET1: SW_Push, Button_Switch_SMD:SW_SPST_TL3342, F.Cu at (257.3, 45.1)
- added U1: ADC108S022CIMTX/NOPB, ADCs:MTC16, B.Cu at (33.5, 64.0)
- added U10: DRV5053VAQDBZR, HallEffect:DBZ0003A_N, B.Cu at (103.2, 63.0)
- added U11: DRV5053VAQDBZR, HallEffect:DBZ0003A_N, B.Cu at (140.2, 66.0)
- added U12: DRV5053VAQDBZR, HallEffect:DBZ0003A_N, B.Cu at (141.2, 102.0)
- added U13: DRV5053VAQDBZR, HallEffect:DBZ0003A_N, B.Cu at (171.5, 88.5)
- added U14: DRV5053VAQDBZR, HallEffect:DBZ0003A_N, B.Cu at (236.0, 72.0)
- added U15: DRV5053VAQDBZR, HallEffect:DBZ0003A_N, B.Cu at (48.5, 74.2)
- added U16: DRV5053VAQDBZR, HallEffect:DBZ0003A_N, B.Cu at (43.6, 60.6)
- added U17: DRV5053VAQDBZR, HallEffect:DBZ0003A_N, B.Cu at (43.6, 65.1)
- added U18: DRV5053VAQDBZR, HallEffect:DBZ0003A_N, B.Cu at (43.6, 69.7)
- added U19: DRV5053VAQDBZR, HallEffect:DBZ0003A_N, B.Cu at (202.7, 79.0)
- added U20: ATmega32U4-A, Package_QFP:TQFP-44_10x10mm_P0.8mm, F.Cu at (265.7, 33.5)
- added U3: ADC108S022CIMTX/NOPB, ADCs:MTC16, B.Cu at (33.5, 70.8)
- added U4: DRV5053VAQDBZR, HallEffect:DBZ0003A_N, B.Cu at (170.5, 52.5)
- added U5: DRV5053VAQDBZR, HallEffect:DBZ0003A_N, B.Cu at (201.7, 43.1)
- added U6: DRV5053VAQDBZR, HallEffect:DBZ0003A_N, B.Cu at (235.0, 36.0)
- added U7: DRV5053VAQDBZR, HallEffect:DBZ0003A_N, B.Cu at (117.7, 130.0)
- added U8: DRV5053VAQDBZR, HallEffect:DBZ0003A_N, B.Cu at (72.9, 49.5)
- added U9: DRV5053VAQDBZR, HallEffect:DBZ0003A_N, B.Cu at (41.7, 40.1)
- added Y2: Crystal_GND24, Crystal:Crystal_SMD_SeikoEpson_FA238-4Pin_3.2x2.5mm, F.Cu at (265.2, 43.0)
- moved D1 127.7 mm to (252.5, 25.0)
- moved D2 127.7 mm to (252.5, 26.8)
- moved C3 50.9 mm to (78.0, 105.5)
- moved C5 50.9 mm to (89.3, 95.6)
- moved C7 50.9 mm to (78.0, 97.3)
- moved C4 50.9 mm to (83.2, 106.0)
- moved C6 50.9 mm to (79.9, 100.5)
- moved C9 50.9 mm to (72.7, 108.5)
- moved R1 50.9 mm to (79.2, 117.0)
- moved R4 50.9 mm to (74.2, 116.5)
- moved R5 50.9 mm to (76.7, 128.5)
Routing:
- net GND: track 14.4 -> 0.00 mm, vias 1 -> 0
- net Net-(U2-XTAL1): track 6.90 -> 0.00 mm
- net Net-(U2-XTAL2): track 6.34 -> 0.00 mm

Commit message: Updated PCB and schematic with the Gateron footprint, added dummy Brooks footprint
Parts:
- added Brooks1: ~, BrooksBoards:BrooksP5Plus, F.Cu at (228.5, 125.0)
- added U2: ~, key-switches:Gateron Jade Pro Magnetic, F.Cu at (41.7, 40.1)
- added U21: ~, key-switches:Gateron Jade Pro Magnetic, F.Cu at (-87.3, 79.3)
- added U22: ~, key-switches:Gateron Jade Pro Magnetic, F.Cu at (-87.3, 94.4)
- added U23: ~, key-switches:Gateron Jade Pro Magnetic, F.Cu at (-87.3, 109.5)
- added U24: ~, key-switches:Gateron Jade Pro Magnetic, F.Cu at (72.9, 49.5)
- added U25: ~, key-switches:Gateron Jade Pro Magnetic, F.Cu at (235.0, 36.0)
- added U26: ~, key-switches:Gateron Jade Pro Magnetic, F.Cu at (236.0, 72.0)
- added U27: ~, key-switches:Gateron Jade Pro Magnetic, F.Cu at (-72.2, 109.5)
- added U28: ~, key-switches:Gateron Jade Pro Magnetic, F.Cu at (103.2, 63.0)
- added U29: ~, key-switches:Gateron Jade Pro Magnetic, F.Cu at (170.5, 52.5)
- added U30: ~, key-switches:Gateron Jade Pro Magnetic, F.Cu at (202.7, 79.0)
- added U31: ~, key-switches:Gateron Jade Pro Magnetic, F.Cu at (201.7, 43.1)
- added U32: ~, key-switches:Gateron Jade Pro Magnetic, F.Cu at (140.2, 66.0)
- added U33: ~, key-switches:Gateron Jade Pro Magnetic, F.Cu at (117.7, 130.0)
- added U34: ~, key-switches:Gateron Jade Pro Magnetic, F.Cu at (141.2, 101.9)
- added U35: ~, key-switches:Gateron Jade Pro Magnetic, F.Cu at (171.5, 88.5)
Routing:
- net GND: track 0.00 -> 80.6 mm
Other:
- board size 302.5 x 158.3 mm -> 259.5 x 132.8 mm

Commit message: Fallback Pico GP2040-CE added
Parts:
- removed C9: 100n, Capacitor_SMD:C_0603_1608Metric
- removed R1: 10k, Resistor_SMD:R_0603_1608Metric
- added ?: , , B.Cu at (31.9, 91.5)
- added ?: , , B.Cu at (53.2, 88.9)
- added U36: ~, BrooksBoards:BrooksP5Mini, F.Cu at (215.5, 123.5)
- added U37: Pico, MCU_RaspberryPi_and_Boards:RPi_Pico_SMD_TH, F.Cu at (261.0, 120.5)
- C10, C11, C3, C4, C5, C6, C7, C8, D2, J1, R10, R2, R3, R5, R6, R7, R9, SW_RESET1, U20, Y2: moved to B.Cu
- moved U23 256.6 mm to (156.7, 30.0)
- moved J1 249.1 mm to (23.0, 97.2), turned to 90 degrees
- moved D2 230.3 mm to (31.5, 91.5), turned to 180 degrees
- moved U20 221.0 mm to (54.5, 98.5)
- moved U27 220.7 mm to (136.3, 37.1)
- moved SW_RESET1 217.1 mm to (44.8, 89.5), turned to -90 degrees
- moved Y2 215.6 mm to (54.5, 88.7), turned to 45 degrees
- moved C10 214.8 mm to (52.5, 86.7), turned to -135 degrees
- moved C8 214.8 mm to (56.5, 86.7), turned to -45 degrees
- moved U22 210.3 mm to (115.0, 37.0)
- moved U21 187.9 mm to (94.0, 30.0)
- moved R4 186.8 mm to (234.2, 20.0)
- moved U1 149.4 mm to (182.8, 68.0), turned to -90 degrees
- moved U15 116.9 mm to (156.7, 30.0)
- moved U18 98.3 mm to (136.3, 37.1)
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Connections:
- U1 pad 10: HKA -> MKA
- U1 pad 11: SHKA -> LKA
- U1 pad 8: LKA -> SHKA
- U1 pad 9: MKA -> HKA
- U3 pad 4: UA -> LA
- U3 pad 6: LA -> RA
- U3 pad 7: RA -> SELECTA
- U3 pad 9: SELECTA -> UA
Routing:
- net VCC: track 0.00 -> 316.6 mm, vias 0 -> 6
- net /L: track 0.00 -> 202.2 mm, vias 0 -> 1
- net /LP: track 0.00 -> 193.0 mm, vias 0 -> 1
- net /HP: track 0.00 -> 191.6 mm, vias 0 -> 1
- net /MP: track 0.00 -> 183.8 mm, vias 0 -> 1
- net /MK: track 0.00 -> 183.6 mm, vias 0 -> 1
- net /SHP: track 0.00 -> 183.6 mm, vias 0 -> 1
- net /LK: track 0.00 -> 183.4 mm, vias 0 -> 1
- net /U: track 0.00 -> 183.2 mm, vias 0 -> 1
- net /D: track 0.00 -> 182.9 mm, vias 0 -> 1
- net /R: track 0.00 -> 182.7 mm, vias 0 -> 1
- net /HK: track 0.00 -> 182.3 mm, vias 0 -> 1
- net /SHK: track 0.00 -> 181.0 mm, vias 0 -> 1
- net NOT_CS1: track 0.00 -> 173.3 mm, vias 0 -> 2
- net SCLK: track 0.00 -> 156.1 mm, vias 0 -> 3
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- added copper zone on B.Cu, net VCC
